File: STM32F401CCT6 KART/STM32F401CCT6.kicad_sch (KiCad schematic)
At the start: 43 parts

Commit message: STM32F042x6 ARM TEMEL KARTI
NOT:KART PINLERI DEGISTIRILDI.!
Parts:
- C1, C2: value (none) -> 22n,0603; footprint (none) -> Capacitors_SMD:C_0603
- C10, C11: value (none) -> 4.7uF,0603; footprint (none) -> Capacitors_SMD:C_0603
- C12, C13, C14, C17, C18, C5: value (none) -> 0.1U,0603; footprint (none) -> Capacitors_SMD:C_0603
- C15: value (none) -> 4.7u,0603; footprint (none) -> Capacitors_SMD:C_0603
- C16, C19: value (none) -> 0.1uF,0603; footprint (none) -> Capacitors_SMD:C_0603
- C3: value (none) -> 1U,0603; footprint (none) -> Capacitors_SMD:C_0603
- C4: value (none) -> 10U,0603; footprint (none) -> Capacitors_SMD:C_0603
- C6, C7, C8, C9: value (none) -> 20p,0603; footprint (none) -> Capacitors_SMD:C_0603
- D1: value (none) -> RED_LED; footprint (none) -> LEDs:LED_0805
- D2: value (none) -> BLUE_LED; footprint (none) -> LEDs:LED_0805
- J1: value (none) -> USB_OTG; footprint (none) -> Connectors_USB:USB_Micro-B_Molex-105017-0001
- J2: value (none) -> Conn_02x03_Odd_Even; footprint (none) -> Pin_Headers:Pin_Header_Straight_2x03_Pitch2.54mm
- J3: value (none) -> Conn_01x20_des; footprint (none) -> Pin_Headers:Pin_Header_Straight_1x20_Pitch2.54mm
- J4: value (none) -> Conn_01x05_desc; footprint (none) -> Pin_Headers:Pin_Header_Angled_1x05_Pitch2.54mm
- J5: value (none) -> Conn_01x20; footprint (none) -> Pin_Headers:Pin_Header_Straight_1x20_Pitch2.54mm
- R1, R11: value (none) -> 10K; footprint (none) -> Resistors_SMD:R_0603
- R10: value (none) -> 4.7K; footprint (none) -> Resistors_SMD:R_0603
- R2: value (none) -> 1M; footprint (none) -> Resistors_SMD:R_0603
- R3, R4, R9: value (none) -> 20R,0603; footprint (none) -> Resistors_SMD:R_0603
- R5: value (none) -> 510R,0603; footprint (none) -> Resistors_SMD:R_0603
- R6: value (none) -> 510R,603; footprint (none) -> Resistors_SMD:R_0603
- R7, R8: value (none) -> 100K,0603; footprint (none) -> Resistors_SMD:R_0603
- SW1: value (none) -> SW_Push; footprint (none) -> Buttons_Switches_SMD:SW_SPST_TL3342
- U1: value (none) -> MIC5219-3.3; footprint (none) -> TO_SOT_Packages_SMD:SOT-23-5
- U2: value (none) -> STM32F401CCT6
- U3: value (none) -> USBLC6-2SC6; footprint (none) -> TO_SOT_Packages_SMD:SOT-23-6
- Y1: value (none) -> 32.786K; footprint (none) -> Crystals:Crystal_SMD_SeikoEpson_MC306-4pin_8.0x3.2mm
- Y2: value (none) -> 8MHz; footprint (none) -> Crystals:Crystal_HC49-4H_Vertical
